File: ISO PCB/southpawpcb.sch (KiCad schematic (older format))
At the start: 160 parts, among them K1 KEYSW, K10 KEYSW, K11 KEYSW, K12 KEYSW, K13 KEYSW, K14 KEYSW, K15 KEYSW, K16 KEYSW, K17 KEYSW, K18 KEYSW, K19 KEYSW, K2 KEYSW, K20 KEYSW, K21 KEYSW, K22 KEYSW, K23 KEYSW, K24 KEYSW, K25 KEYSW, K26 KEYSW, K27 KEYSW, K28 KEYSW, K29 KEYSW, K3 KEYSW, K30 KEYSW, K31 KEYSW, K32 KEYSW, K33 KEYSW, K34 KEYSW, K35 KEYSW, K36 KEYSW, K37 KEYSW, K38 KEYSW, K39 KEYSW, K4 KEYSW, K40 KEYSW, K41 KEYSW, K42 KEYSW, K43 KEYSW, K44 KEYSW, K45 KEYSW, K46 KEYSW, K47 KEYSW, K48 KEYSW, K49 KEYSW, K5 KEYSW, K50 KEYSW, K51 KEYSW, K52 KEYSW, K53 KEYSW, K54 KEYSW, K55 KEYSW, K56 KEYSW, K57 KEYSW, K58 KEYSW, K59 KEYSW, K6 KEYSW, K60 KEYSW, K61 KEYSW, K62 KEYSW, K63 KEYSW, K64 KEYSW, K65 KEYSW, K66 KEYSW, K67 KEYSW, K68 KEYSW, K69 KEYSW, K7 KEYSW, K70 KEYSW, K71 KEYSW, K72 KEYSW, K73 KEYSW, K74 KEYSW, K75 KEYSW, K76 KEYSW, K77 KEYSW, K78 KEYSW, K79 KEYSW, K8 KEYSW, K9 KEYSW, SW1 Reset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

Commit message: Fixing missing libraries, redrawing schematic
Parts:
- removed D79: D, Canadian_Footprints:D_SOD123_axial-dual, symbol Device:D
- removed K1, K10, K11, K12, K13, K14, K15, K16, K17, K19, K2, K20, K21, K24, K25, K26, K27, K28, K29, K3, K30, K31, K32, K33, K34, K35, K37, K38, K39, K4, K41, K42, K43, K44, K45, K46, K47, K48, K49, K5, K50, K51, K52, K53, K54, K55, K58, K59, K6, K60, K61, K62, K63, K64, K65, K66, K67, K68, K7, K71, K8, K9: KEYSW, MX/Alps_Hybrid:MX-1U-NoLED, symbol Keyboard_Parts1:KEYSW
- removed K18, K22, K56, K70: KEYSW, MX/Alps_Hybrid:MX-2U-NoLED, symbol Keyboard_Parts1:KEYSW
- removed K23: KEYSW, MX/Alps_Hybrid:MX-1.5U-NoLED, symbol Keyboard_Parts1:KEYSW
- removed K36: KEYSW, MX/Alps_Hybrid:MX-ISO, symbol Keyboard_Parts1:KEYSW
- removed K40: KEYSW, MX/Alps_Hybrid:MX-1.75U-NoLED, symbol Keyboard_Parts1:KEYSW
- removed K57, K72, K73, K74, K76, K77, K78, K79: KEYSW, MX/Alps_Hybrid:MX-1.25U-NoLED, symbol Keyboard_Parts1:KEYSW
- removed K69: KEYSW, MX/Alps_Hybrid:MX-2.75U-NoLED, symbol Keyboard_Parts1:KEYSW
- removed K75: KEYSW, MX/Alps_Hybrid:MX-6.25U-NoLED, symbol Keyboard_Parts1:KEYSW
- removed SW1: Reset, Button_Switch_SMD:SW_SPST_TL3342, symbol Keyboard_Parts1:SW_PUSH
- removed U1: ProMicro, Pro_Micro:ProMicro, symbol Pro_Micro:ProMicro
- added K1, K10, K11, K12, K13, K14, K15, K16, K17, K18, K19, K2, K20, K21, K22, K23, K24, K25, K26, K27, K28, K29, K3, K30, K31, K32, K33, K34, K35, K36, K37, K38, K39, K4, K40, K41, K42, K43, K44, K45, K46, K47, K48, K49, K5, K50, K51, K52, K53, K54, K55, K56, K57, K58, K59, K6, K60, K61, K62, K63, K64, K65, K66, K67, K68, K69, K7, K70, K71, K72, K73, K74, K75, K76, K77, K78, K8, K9: KEYSW, symbol KeyboardParts:KEYSW
- added SW1: Reset, symbol Switch:SW_Push
- added U1: ProMicro, symbol ProMicro:ProMicro
- D1, D10, D11, D12, D13, D14, D15, D16, D17, D18, D19, D2, D20, D21, D22, D23, D24, D25, D26, D27, D28, D29, D3, D30, D31, D32, D33, D34, D35, D36, D37, D38, D39, D4, D40, D41, D42, D43, D44, D45, D46, D47, D48, D49, D5, D50, D51, D52, D53, D54, D55, D56, D57, D58, D59, D6, D60, D61, D62, D63, D64, D65, D66, D67, D68, D69, D7, D70, D71, D72, D73, D74, D75, D76, D77, D78, D8, D9: footprint Canadian_Footprints:D_SOD123_axial-dual -> (none)
Connections:
- wire segments 189 -> 217
